Commit message: Changes to improve performance -Raised effort and velocity limits -Recalibration of PID controllers explained in pid_calib file

File: thor_description/urdf/thor_calibration.xacro (robot description, xacro)
@@ -17,12 +17,12 @@
     <link name ='bar_link'>
       <inertial>
-        <mass value="0.15"/>
+        <mass value="0.5"/>
         <inertia
-          ixx="1.506666E-3"
+          ixx="3.766666E-3"
           ixy="0"
           ixz="0"
-          iyy="1.506666E-3"
+          iyy="3.766666E-3"
           iyz="0"
-          izz="1.333333E-5"/>
+          izz="3.333333E-5"/>
       </inertial>
       <collision name="collision">

File: thor_description/urdf/thor_description.urdf.xacro (robot description, xacro)
@@ -7,6 +7,6 @@
 <robot xmlns:xacro="http://wiki.ros.org/xacro">
   <xacro:property name="damping" value="0.01" /> <!-- Joint Damping -->
-  <xacro:property name="effort_limit" value="10" />  <!-- Maximum Torque -->
-  <xacro:property name="velocity_limit" value="2" />  <!-- Maximum Joint Velocity -->
+  <xacro:property name="effort_limit" value="100" />  <!-- Maximum Torque -->
+  <xacro:property name="velocity_limit" value="10" />  <!-- Maximum Joint Velocity -->
   <!-- MAIN MACRO: Generates the URDF of the THOR Robot-->
   <xacro:macro name="thor_robot" params="prefix">
